Commit message: marco : added param to run ros control gazebo

File: schunk_gazebo/urdf/gazebo_complete.xacro (robot description, xacro)
@@ -1,5 +1,5 @@
 <?xml version="1.0"?>
 <robot xmlns:xacro="http://ros.org/wiki/xacro" name="egk_40">
-  <xacro:macro name="egk_40_gazebo" params="prefix parent px py pz rx ry rz hardware_interface">
+  <xacro:macro name="egk_40_gazebo" params="prefix parent px py pz rx ry rz hardware_interface launch_gazebo_ros_control_plugin='yes'">
     <!-- includes -->
     <xacro:include filename="$(find schunk_description)/urdf/egk_40_complete.xacro" />
@@ -15,10 +15,12 @@
     <xacro:egk_40_transmission hardware_interface="${hardware_interface}" />
     <!-- Loading Gazebo plugins -->
-    <gazebo>
-      <plugin name="ros_control" filename="libgazebo_ros_control.so">
-        <!--robotNamespace>/</robotNamespace-->
-        <!--robotSimType>gazebo_ros_control/DefaultRobotHWSim</robotSimType-->
-      </plugin>
-    </gazebo>
+    <xacro:if value="${launch_gazebo_ros_control_plugin == 'yes'}">
+      <gazebo>
+        <plugin name="ros_control" filename="libgazebo_ros_control.so">
+          <!--robotNamespace>/</robotNamespace-->
+          <!--robotSimType>gazebo_ros_control/DefaultRobotHWSim</robotSimType-->
+        </plugin>
+      </gazebo>
+    </xacro:if>
     <!-- Disabling gravity -->
     <gazebo reference="finger1">

Commit message: marco : changed yes/no to true/false

File: schunk_gazebo/urdf/gazebo_complete.xacro (robot description, xacro)
@@ -1,5 +1,5 @@
 <?xml version="1.0"?>
 <robot xmlns:xacro="http://ros.org/wiki/xacro" name="egk_40">
-  <xacro:macro name="egk_40_gazebo" params="prefix parent px py pz rx ry rz hardware_interface launch_gazebo_ros_control_plugin='yes'">
+  <xacro:macro name="egk_40_gazebo" params="prefix parent px py pz rx ry rz hardware_interface launch_gazebo_ros_control_plugin='true'">
     <!-- includes -->
     <xacro:include filename="$(find schunk_description)/urdf/egk_40_complete.xacro" />
@@ -15,5 +15,5 @@
     <xacro:egk_40_transmission hardware_interface="${hardware_interface}" />
     <!-- Loading Gazebo plugins -->
-    <xacro:if value="${launch_gazebo_ros_control_plugin == 'yes'}">
+    <xacro:if value="${launch_gazebo_ros_control_plugin}">
       <gazebo>
         <plugin name="ros_control" filename="libgazebo_ros_control.so">
