Commit message: Created test for schunk_description

File: schunk_description/urdf/egk_40_complete.xacro (robot description, xacro)
@@ -1,29 +1,17 @@
 <?xml version="1.0"?>
 <robot xmlns:xacro="http://ros.org/wiki/xacro" name="egk_40_complete" >
-  <!-- parameters -->
-  <xacro:arg name="prefix" default=""/>
-  <xacro:arg name="parent" default="world"/>
-  <xacro:property name="parent" value="$(arg parent)" />
-  <xacro:arg name="px" default="0.0"/>
-  <xacro:arg name="py" default="0.0"/>
-  <xacro:arg name="pz" default="0.0"/>
-  <xacro:arg name="rx" default="0.0"/>
-  <xacro:arg name="ry" default="0.0"/>
-  <xacro:arg name="rz" default="0.0"/>
-  <!-- includes -->
-  <xacro:include filename="$(find schunk_description)/urdf/egk_40.xacro" />
-  <!-- define world link -->
-  <xacro:if value="${parent == 'world'}">
-    <link name="world" />
-  </xacro:if>
-  <!-- Gripper's main body -->
-  <xacro:egk_40 prefix="$(arg prefix)"/>
-  <!-- Fingers -->
-  <!-- TODO -->
-  <!-- Joint connecting gripper base (gripper_body) to parent -->
-  <joint name="parent_to_gripper" type="fixed">
-    <parent link="$(arg parent)" />
-    <child  link="$(arg prefix)gripper_body" />
-    <origin xyz="$(arg px) $(arg py) $(arg pz)" rpy="$(arg rx) $(arg ry) $(arg rz)" />
-  </joint>
+  <xacro:macro name="egk_40_complete" params="prefix parent px py pz rx ry rz">
+    <!-- includes -->
+    <xacro:include filename="$(find schunk_description)/urdf/egk_40.xacro" />
+    <!-- Gripper's main body -->
+    <xacro:egk_40 prefix="$(arg prefix)"/>
+    <!-- Fingers -->
+    <!-- TODO -->
+    <!-- Joint connecting gripper base (gripper_body) to parent -->
+    <joint name="parent_to_gripper" type="fixed">
+      <parent link="$(arg parent)" />
+      <child  link="$(arg prefix)gripper_body" />
+      <origin xyz="$(arg px) $(arg py) $(arg pz)" rpy="$(arg rx) $(arg ry) $(arg rz)" />
+    </joint>
+  </xacro:macro>
 </robot>

Commit message: Possible to lauch gripper gazebo outside of pkg itself

File: schunk_description/urdf/egk_40_complete.xacro (robot description, xacro)
@@ -5,12 +5,12 @@
     <xacro:include filename="$(find schunk_description)/urdf/egk_40.xacro" />
     <!-- Gripper's main body -->
-    <xacro:egk_40 prefix="$(arg prefix)"/>
+    <xacro:egk_40 prefix="${prefix}"/>
     <!-- Fingers -->
     <!-- TODO -->
     <!-- Joint connecting gripper base (gripper_body) to parent -->
     <joint name="parent_to_gripper" type="fixed">
-      <parent link="$(arg parent)" />
-      <child  link="$(arg prefix)gripper_body" />
-      <origin xyz="$(arg px) $(arg py) $(arg pz)" rpy="$(arg rx) $(arg ry) $(arg rz)" />
+      <parent link="${parent}" />
+      <child  link="${prefix}gripper_body" />
+      <origin xyz="${px} ${py} ${pz}" rpy="${rx} ${ry} ${rz}" />
     </joint>
   </xacro:macro>

File: schunk_gazebo/urdf/gazebo_complete.xacro (robot description, xacro)
@@ -8,10 +8,10 @@
     <!-- Gripper's main body -->
     <xacro:egk_40_complete
-      prefix="$(arg prefix)"
-      parent="$(arg parent)"
-      px="$(arg px)" py="$(arg py)" pz="$(arg pz)"
-      rx="$(arg rx)" ry="$(arg ry)" rz="$(arg rz)" />
+      prefix="${prefix}"
+      parent="${parent}"
+      px="${px}" py="${py}" pz="${pz}"
+      rx="${rx}" ry="${ry}" rz="${rz}" />
     <!-- Tramsmissions -->
-    <xacro:egk_40_transmission hardware_interface="$(arg hardware_interface)" />
+    <xacro:egk_40_transmission hardware_interface="${hardware_interface}" />
     <!-- Loading Gazebo plugins -->
     <gazebo>
