Commit message: Added inertial terms to xacro

File: schunk_description/urdf/egk_40.xacro (robot description, xacro)
@@ -27,4 +27,12 @@
         </geometry>
       </collision>
+      <inertial>
+        <origin xyz="0 0 0" rpy="0 0 0" />
+        <mass value="1.5" />
+        <inertia
+          ixx="1.0" ixy="0.0" ixz="0.0"
+          iyy="1.0" iyz="0.0"
+          izz="1.0" />
+      </inertial>
     </link>
     <!-- Finger 1 -->
@@ -45,4 +53,12 @@
         </geometry>
       </collision>
+      <inertial>
+        <origin xyz="0 0 0" rpy="0 0 0" />
+        <mass value="0.1" />
+        <inertia
+          ixx="0.001" ixy="0.0" ixz="0.0"
+          iyy="0.001" iyz="0.0"
+          izz="0.001" />
+      </inertial>
     </link>
     <!-- Finger 2 -->
@@ -63,7 +79,15 @@
         </geometry>
       </collision>
+      <inertial>
+        <origin xyz="0 0 0" rpy="0 0 0" />
+        <mass value="0.1" />
+        <inertia
+          ixx="0.001" ixy="0.0" ixz="0.0"
+          iyy="0.001" iyz="0.0"
+          izz="0.001" />
+      </inertial>
     </link>
     <!-- joints: main serial chain -->
-    <joint name="${prefix}gripper_body-finger1" type="prismatic">
+    <joint name="${prefix}finger1_joint" type="prismatic">
       <parent link="${prefix}gripper_body" />
       <child link="${prefix}finger1" />
@@ -71,5 +95,5 @@
       <limit lower="0.0" upper="0.04" effort="100.0" velocity="10.0" />
     </joint>
-    <joint name="${prefix}gripper_body-finger2" type="prismatic">
+    <joint name="${prefix}finger2_joint" type="prismatic">
       <parent link="${prefix}gripper_body" />
       <child link="${prefix}finger2" />

Commit message: Fixed joint limits

File: schunk_description/urdf/egk_40.xacro (robot description, xacro)
@@ -93,5 +93,5 @@
       <child link="${prefix}finger1" />
       <origin xyz="0.016 0.071 0.02" rpy="0 ${pi/2} 0" />
-      <limit lower="0.0" upper="0.04" effort="100.0" velocity="10.0" />
+      <limit lower="0.0" upper="0.0415" effort="100.0" velocity="10.0" />
     </joint>
     <joint name="${prefix}finger2_joint" type="prismatic">
@@ -99,5 +99,5 @@
       <child link="${prefix}finger2" />
       <origin xyz="-0.016 0.071 -0.02" rpy="0 ${-pi/2} 0" />
-      <limit lower="0.0" upper="0.04" effort="100.0" velocity="10.0" />
+      <limit lower="0.0" upper="0.0415" effort="100.0" velocity="10.0" />
     </joint>
   </xacro:macro>

Commit message: PID tuning + change physical params

File: schunk_description/urdf/egk_40.xacro (robot description, xacro)
@@ -55,9 +55,9 @@
       <inertial>
         <origin xyz="0 0 0" rpy="0 0 0" />
-        <mass value="0.1" />
+        <mass value="0.3" />
         <inertia
-          ixx="0.001" ixy="0.0" ixz="0.0"
-          iyy="0.001" iyz="0.0"
-          izz="0.001" />
+          ixx="0.1" ixy="0.0" ixz="0.0"
+          iyy="0.1" iyz="0.0"
+          izz="0.1" />
       </inertial>
     </link>
@@ -81,9 +81,9 @@
       <inertial>
         <origin xyz="0 0 0" rpy="0 0 0" />
-        <mass value="0.1" />
+        <mass value="0.3" />
         <inertia
-          ixx="0.001" ixy="0.0" ixz="0.0"
-          iyy="0.001" iyz="0.0"
-          izz="0.001" />
+          ixx="0.1" ixy="0.0" ixz="0.0"
+          iyy="0.1" iyz="0.0"
+          izz="0.1" />
       </inertial>
     </link>
@@ -93,5 +93,5 @@
       <child link="${prefix}finger1" />
       <origin xyz="0.016 0.071 0.02" rpy="0 ${pi/2} 0" />
-      <limit lower="0.0" upper="0.0415" effort="100.0" velocity="10.0" />
+      <limit lower="0.0" upper="0.0415" effort="1000.0" velocity="10.0" />
     </joint>
     <joint name="${prefix}finger2_joint" type="prismatic">
@@ -99,5 +99,5 @@
       <child link="${prefix}finger2" />
       <origin xyz="-0.016 0.071 -0.02" rpy="0 ${-pi/2} 0" />
-      <limit lower="0.0" upper="0.0415" effort="100.0" velocity="10.0" />
+      <limit lower="0.0" upper="0.0415" effort="1000.0" velocity="10.0" />
     </joint>
   </xacro:macro>

Commit message: Changed visual to .dae

File: schunk_description/urdf/egk_40.xacro (robot description, xacro)
@@ -15,5 +15,5 @@
         <origin xyz="0 0 0" rpy="0 0 0" />
         <geometry>
-          <mesh filename="package://schunk_description/meshes/egk40/visual/egk40_body.stl"
+          <mesh filename="package://schunk_description/meshes/egk40/visual/egk40_body.dae"
             scale="0.001 0.001 0.001" />
         </geometry>
@@ -41,5 +41,5 @@
         <origin xyz="0 0 0" rpy="0 0 0" />
         <geometry>
-          <mesh filename="package://schunk_description/meshes/egk40/visual/slider.stl"
+          <mesh filename="package://schunk_description/meshes/egk40/visual/slider.dae"
             scale="0.001 0.001 0.001" />
         </geometry>
@@ -67,5 +67,5 @@
         <origin xyz="0 0 0" rpy="0 0 0" />
         <geometry>
-          <mesh filename="package://schunk_description/meshes/egk40/visual/slider.stl"
+          <mesh filename="package://schunk_description/meshes/egk40/visual/slider.dae"
             scale="0.001 0.001 0.001" />
         </geometry>

File: schunk_description/urdf/finger.xacro (robot description, xacro)
@@ -11,5 +11,5 @@
         <origin xyz="0 0 0" rpy="0 0 0" />
         <geometry>
-          <mesh filename="package://schunk_description/meshes/fingers/visual/flat_finger.stl"
+          <mesh filename="package://schunk_description/meshes/fingers/visual/flat_finger.dae"
             scale="0.001 0.001 0.001" />
         </geometry>
